File: Hardware/Talon_I2C.brd (EAGLE design)
At the start: 140 x 19 mm, 88 parts, among them J1 CONN_TALON_REMOTE, J2 CONN_SDI-12_LOGGERM8_TE_BOARD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, J3 CONN_SDI-12_LOGGERM8_TE_BOARD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, J4 CONN_SDI-12_LOGGERM8_TE_BOARD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, J5 CONN_APOGEE_LOGGER, Q1 AO3419, Q2 2N7002, Q3 AO3419, Q4 2N7002, Q5 AO3419, Q6 2N7002, Q7 AO3419, Q8 2N7002, U1 SN74LVC1G00SC70, U10 SN74LVC1G3157SC70, U11 SN74LVC1G3157SC70, U12 SN74LVC1G3157SC70, U13 SN74LVC1G3157SC70, U14 LM2621, U15 MCP3221, U16 LMR62014SOT23, U17 TXS0102DCU, U18 FDC6330L, U2 SN74LVC2G241DCU, U26 MCP23018QFN, U28 74HC4852, U29 SN74AUP1T157DCK, U3 MAX9034TSSOP, U30 MCP3421A3, U31 PCA9536DFN, U4 INA4180A2, U5 CD4044, U6 SN74HC04, U7 SN74AC08, U8 SIP32431TDFN, U9 SN74LVC1G17DCK

Commit message: Copper layout done
Parts:
- removed C14: 10uF, bschulz_passives:C0805
- removed C15: 220pF, bschulz_passives:C0603
- removed C16: 0.1uF, bschulz_passives:C0603
- removed D2: CDBA3100, bschulz:DO214AC
- removed D4: (no value), bschulz:SOD-123
- removed J2, J3, J4: CONN_SDI-12_LOGGERM8_TE_BOARDLOCK, GEMS_Plugs:1X03_M8_TE_T40410_BOARDLOCK
- removed J5: CONN_APOGEE_LOGGER, GEMS_Plugs:1X06_M8_PHOENIX_1456022_BOARDLOCK
- removed L1: 6.8uH, bschulz:WE-MAIA(4.1X4.1)
- removed L3: 10uH, bschulz:1008
- removed R27, R28: 100k, bschulz_passives:R0603
- removed R31: 40.2k, bschulz_passives:R0603
- removed R32: 13.3k, bschulz_passives:R0603
- removed U1: SN74LVC1G00SC70, bschulz:DCK_R-PDSO-G5
- removed U10: SN74LVC1G3157SC70, bschulz:DCK_R-PDSO-G6
- removed U2: SN74LVC2G241DCU, bschulz:DCU_(R-PDSO-G8)
- removed U9: SN74LVC1G17DCK, bschulz:DCK_R-PDSO-G5
- added J6, J7, J8, J9: CONN_I2C_LOGGER, GEMS_Plugs:1X04_M8_TE_T404103_BOARDLOCK
- added U19, U20: PCA9617WSON, bschulz:WSON-8_2X3
- C1, C10, C12, C3, C6, C8: device bschulz_passives:C0603 -> bschulz_passives:C0402
- C11: value 4.7uF -> 0.1uF; device bschulz_passives:C0805 -> bschulz_passives:C0402
- C2: value 22uF -> 0.1uF; device bschulz_passives:C0805 -> bschulz_passives:C0402
- C4: value (none) -> 0.1uF; device bschulz_passives:C0603 -> bschulz_passives:C0402
- C5: value 68uF -> 0.1uF; device bschulz_passives:C2917 -> bschulz_passives:C0402
- C9: value 10uF -> 0.1uF; device bschulz_passives:C0805 -> bschulz_passives:C0402
- R1, R11, R13, R14, R15, R17, R18, R19, R20, R23, R3, R4, R5, R6, R8, R9: device bschulz_passives:R0603 -> bschulz_passives:R0402
- R16: value (none) -> 100k; device bschulz_passives:R0603 -> bschulz_passives:R0402
- R24: value 470k -> (none); device bschulz_passives:R0603 -> bschulz_passives:R0402
- R25: value 115k -> (none); device bschulz_passives:R0603 -> bschulz_passives:R0402
- R26: value 13.3k -> (none); device bschulz_passives:R0603 -> bschulz_passives:R0402
- U11: value SN74LVC1G3157SC70 -> 24AA02SOT23; device bschulz:DCK_R-PDSO-G6 -> bschulz:SOT23-5
- U12, U13: value SN74LVC1G3157SC70 -> SN74AUP1G08DCK; device bschulz:DCK_R-PDSO-G6 -> bschulz:DCK_R-PDSO-G5
- U14: value LM2621 -> SN74AUP1G08DCK; device bschulz:DGK_S-PDSO-G8 -> bschulz:DCK_R-PDSO-G5
- U15: value MCP3221 -> SN74AUP1G08DCK; device bschulz:SOT23-5 -> bschulz:DCK_R-PDSO-G5
- U16: value LMR62014SOT23 -> FXMAR2102UMLP; device bschulz:DBV0005A -> bschulz:UQFN-8_1.4X1.2
- U17: value TXS0102DCU -> PCA9617WSON; device bschulz:DCU_(R-PDSO-G8) -> bschulz:WSON-8_2X3
- U18: value FDC6330L -> PCA9617WSON; device bschulz:SOT23-6L -> bschulz:WSON-8_2X3
- moved R20 113.0 mm to (-57.4, 8.00), turned to 270 degrees
- moved U17 100.4 mm to (-53.3, 8.00)
- moved C2 86.5 mm to (-55.1, 8.00), turned to 90 degrees
- moved U13 86.1 mm to (-26.4, 8.64)
- moved R19 82.4 mm to (-56.3, 8.00), turned to 270 degrees
- moved R23 77.0 mm to (-18.8, 7.75), turned to 270 degrees
- moved U12 70.3 mm to (-49.5, 7.24)
- moved U18 65.1 mm to (-17.1, 7.87), turned to 180 degrees
- moved C1 57.8 mm to (-51.7, 6.86), turned to 90 degrees
- moved C3 57.0 mm to (-19.8, 5.59), turned to 180 degrees
- moved R24 52.0 mm to (-16.8, 4.70), turned to 0 degrees
- moved C4 51.0 mm to (-19.9, 7.75)
- moved R14 47.4 mm to (-5.71, 6.86), turned to 90 degrees
- moved R15 43.7 mm to (-6.86, 8.13), turned to 270 degrees
- moved R17 40.4 mm to (23.6, 7.62), turned to 270 degrees
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Connections:
- removed net !RX: U2.6, U9.2
- removed net 12V: C4.1, C5.+, D2.C, Q1.2, Q3.2, Q5.2, Q7.2, R1.2, R11.2, R25.2, R27.2, R6.2, R9.2, U18.4
- removed net 5V: C14.1, C15.1, C16.1, C6.1, C9.1, D4.CAT, R31.2, U10.5, U11.5, U12.5, U13.5, U15.1, U17.7, U2.8
- removed net DATA: U10.1, U11.1, U12.1, U13.1, U2.2, U2.3
- removed net DATA_EN1: U10.6, U26.19
- removed net DATA_EN2: U11.6, U26.20
- removed net DATA_EN3: U12.6, U26.21
- removed net DATA_EN4: R28.2, U13.6, U18.5, U26.22
- removed net DATA_OUT1: J2.4, U10.4
- removed net DATA_OUT2: J3.4, U11.4
- removed net DATA_OUT3: J4.4, U12.4
- removed net DATA_OUT4: J5.3, U13.4
- removed net DATA_SENSE4: U13.3, U15.3
- removed net DIR: U2.1, U2.7, U26.7
- removed net FOUT: U1.1, U26.6
- removed net N$10: C15.2, R31.1, R32.2, U16.3
- removed net N$11: R27.1, U18.6
- removed net N$18: U28.3, U29.3
- removed net N$7: C3.2, R24.1, U14.3
- removed net N$8: D2.A, L1.P$2, U14.8
- removed net N$9: C4.2, R25.1, R26.2, U14.4
- removed net RX: J1.1, U9.4
- removed net SCL_HV: U15.5, U17.1
- removed net SDA_HV: U15.4, U17.8
- removed net SW1: D4.ANODE, L3.2, U16.1
- removed net TX: J1.2, U1.2
- removed net VHEATER: J5.5, U18.2, U18.3
- removed net VPORT1_OUT_SENSE: R14.2, R15.2, U28.1
- removed net VPORT2_OUT_SENSE: R16.2, R17.2, U28.5
- removed net VPORT3_OUT_SENSE: R18.2, R19.2, U28.2
- removed net VPORT4_OUT_SENSE: R20.2, R23.2, U28.4
- new net !I2C_OB_EN: U12.1, U13.1, U14.1, U15.1, U6.10
- new net DATA1_EN: U12.2, U26.19
- new net DATA1_EN_LOCAL: U12.4, U17.3
- new net DATA2_EN: U13.2, U26.20
- new net DATA2_EN_LOCAL: U13.4, U18.3
- new net DATA3_EN: U14.2, U26.21
- new net DATA3_EN_LOCAL: U14.4, U19.3
- new net DATA4_EN: U15.2, U26.22
- new net DATA4_EN_LOCAL: U15.4, U20.3
- new net I2C_OB_EN: J1.1, R16.1, U16.5, U6.11
- new net INTB: J1.2, U26.13
- new net N$6: R14.2, R15.1, U29.3
- new net PORT1_SCL: J6.4, R20.1, U17.5
- new net PORT1_SDA: J6.2, R19.1, U17.4
- new net PORT2_SCL: J7.4, R24.1, U18.5
- new net PORT2_SDA: J7.2, R23.1, U18.4
- new net PORT3_SCL: J8.4, R18.1, U19.5
- new net PORT3_SDA: J8.2, R17.1, U19.4
- new net PORT4_SCL: J9.4, R26.1, U20.5
- new net PORT4_SDA: J9.2, R25.1, U20.4
- new net SCL_OB: U11.1, U16.6, U26.9, U30.3, U31.6
- new net SDA_OB: U11.3, U16.7, U26.10, U30.4, U31.7
- net 3V3: now also C5.1, C9.1, Q1.2, Q3.2, Q5.2, Q7.2, R1.2, R11.2, R16.2, R6.2, R9.2, U11.4, U12.5, U13.5, U14.5, U15.5, U16.1, U16.8, U17.7, U18.7, U19.7, U20.7; no longer C10.1, C2.1, L1.P$1, L3.1, R24.2, U1.5, U14.2, U14.6, U14.7, U16.4, U16.5, U17.3, U17.6, U6.11, U9.5
- net GND: now also C3.2, C4.2, C5.2, J6.3, J7.3, J8.3, J9.3, R14.1, U11.5, U12.3, U13.3, U14.3, U15.3, U16.4, U17.EP, U18.2, U18.EP, U19.2, U19.EP, U20.2, U20.EP; no longer C14.2, C16.2, C5.-, J2.3, J3.3, J4.3, J5.1, J5.6, R15.1, R17.1, R19.1, R23.1, R26.1, R28.1, R32.1, U1.3, U10.2, U12.2, U13.2, U14.1, U14.5, U15.2, U16.2, U18.1, U2.4, U9.3
- net N$5: now also R15.2, U28.3; no longer U1.4, U2.5
- net SCL: now also U16.3, U17.8, U18.8, U19.8, U20.8; no longer U17.4, U26.9, U30.3, U31.6
- net SDA: now also U16.2, U17.1, U18.1, U19.1, U20.1; no longer U17.5, U26.10, U30.4, U31.7
- net VPORT1_OUT: now also C2.1, J6.1, R19.2, R20.2, U17.6, U28.1; no longer J2.1, R14.1
- net VPORT2_OUT: now also C4.1, J7.1, R23.2, R24.2, U18.6, U28.5; no longer J3.1, R16.1
- net VPORT3_OUT: now also C6.1, J8.1, R17.2, R18.2, U19.6, U28.2; no longer J4.1, R18.1
- net VPORT4_OUT: now also C10.1, J9.1, R25.2, R26.2, U20.6, U28.4; no longer J5.2, R20.1
Routing:
- net 5V: track 187.7 -> 0.00 mm, vias 6 -> 0
- net DATA: track 179.0 -> 0.00 mm, vias 5 -> 0
- net 12V: track 160.8 -> 0.00 mm, vias 5 -> 0
- net 3V3: track 210.9 -> 354.7 mm, vias 8 -> 14
- net DATA_EN4: track 129.3 -> 0.00 mm, vias 5 -> 0
- net !I2C_OB_EN: track 0.00 -> 125.2 mm, vias 0 -> 5
- net DATA4_EN: track 0.00 -> 88.1 mm, vias 0 -> 2
- net VPORT1_OUT: track 53.1 -> 135.5 mm, vias 0 -> 3
- net VPORT4_OUT: track 114.4 -> 189.3 mm, vias 3 -> 5
- net VPORT4_OUT_SENSE: track 72.7 -> 0.00 mm, vias 2 -> 0
- net DATA3_EN: track 0.00 -> 69.7 mm, vias 0 -> 2
- net DATA_EN3: track 59.0 -> 0.00 mm, vias 2 -> 0
- net VPORT1_OUT_SENSE: track 57.0 -> 0.00 mm, vias 4 -> 0
- net DIR: track 51.1 -> 0.00 mm, vias 2 -> 0
- net DATA_EN1: track 43.2 -> 0.00 mm, vias 2 -> 0
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- removed copper zone on layer 1, net 12V
- removed copper zone on layer 1, net 3V3
- removed copper zone on layer 1, net 5V
- removed copper zone on layer 1, net GND
- removed copper zone on layer 16, net GND
- removed copper zone on layer 1, net N$8
- removed copper zone on layer 1, net SW1

Commit message: Generated gerbers for v0.0
Ready for final review
Parts:
- removed U26: MCP23018QFN, bschulz:QFN24
- removed U29: SN74AUP1T157DCK, bschulz:DCK_R-PDSO-G6
- removed U30: MCP3421A3, bschulz:SOT23-6L
- added U1: SN74HC04, bschulz:TSSOP14
- added U2: CD4044, bschulz:TSSOP16
- added U21: SN74AUP1G08DCK, bschulz:DCK_R-PDSO-G5
- C1: value 0.1uF -> 1uF; device bschulz_passives:C0402 -> bschulz_passives:C0603
- C13: value 10uF -> 0.1uF; device bschulz_passives:C0805 -> bschulz_passives:C0402
- C4: value 0.1uF -> 10uF; device bschulz_passives:C0402 -> bschulz_passives:C0805
- C7: value 1uF -> 0.1uF; device bschulz_passives:C0603 -> bschulz_passives:C0402
- Q1, Q3: value AO3419 -> 2N7002
- Q6, Q8: value 2N7002 -> AO3419
- R10, R2: value 82m -> 10k; device bschulz_passives:R0603 -> bschulz_passives:R0402
- R11: value 10k -> 1M
- R12: value 82m -> 100k; device bschulz_passives:R0603 -> bschulz_passives:R0402
- R13: value 100k -> (none); device bschulz_passives:R0402 -> bschulz_passives:R0603
- R14: device bschulz_passives:R0402 -> bschulz_passives:R0603
- R16: value 100k -> (none)
- R17, R18, R19, R20, R23, R24, R25, R26: value (none) -> 10k
- R21, R22: value (none) -> 10k; device bschulz_passives:R0603 -> bschulz_passives:R0402
- R5: value 1M -> 82m; device bschulz_passives:R0402 -> bschulz_passives:R0603
- R6, R8: value 10k -> 82m; device bschulz_passives:R0402 -> bschulz_passives:R0603
- R9: value 10k -> 100k
- U11: value 24AA02SOT23 -> SN74AUP1T157DCK; device bschulz:SOT23-5 -> bschulz:DCK_R-PDSO-G6
- U12: value SN74AUP1G08DCK -> MCP3421A3; device bschulz:DCK_R-PDSO-G5 -> bschulz:SOT23-6L
- U13: value SN74AUP1G08DCK -> FXMAR2102UMLP; device bschulz:DCK_R-PDSO-G5 -> bschulz:UQFN-8_1.4X1.2
- U14, U15: value SN74AUP1G08DCK -> PCA9617WSON; device bschulz:DCK_R-PDSO-G5 -> bschulz:WSON-8_2X3
- U16: value FXMAR2102UMLP -> PCA9617WSON; device bschulz:UQFN-8_1.4X1.2 -> bschulz:WSON-8_2X3
- U18, U19, U20: value PCA9617WSON -> SN74AUP1G08DCK; device bschulz:WSON-8_2X3 -> bschulz:DCK_R-PDSO-G5
- U3: value MAX9034TSSOP -> SIP32431TDFN; device bschulz:TSSOP14 -> bschulz:TDFN_4
- U5: value CD4044 -> MAX9034TSSOP; device bschulz:TSSOP16 -> bschulz:TSSOP14
- U6: value SN74HC04 -> SN74AC08
- U7: value SN74AC08 -> 24AA02SOT23; device bschulz:TSSOP14 -> bschulz:SOT23-5
- U8: value SIP32431TDFN -> MCP23018QFN; device bschulz:TDFN_4 -> bschulz:QFN24
- moved R1 108.7 mm to (-53.1, 4.83)
- moved R8 107.2 mm to (53.1, 5.71)
- moved U17 100.4 mm to (46.7, 16.0), turned to 0 degrees
- moved C9 97.3 mm to (-51.7, 6.86), turned to 90 degrees
- moved U14 83.5 mm to (-53.3, 8.00), turned to 180 degrees
- moved R22 80.9 mm to (51.2, 16.0)
- moved Q5 76.7 mm to (-53.8, 2.29)
- moved R7 76.7 mm to (21.1, 4.57)
- moved Q4 75.5 mm to (58.0, 4.57)
- moved R2 72.9 mm to (-19.8, 4.19), turned to 180 degrees
- moved C10 69.3 mm to (-19.9, 7.75), turned to 90 degrees
- moved U15 63.8 mm to (-17.1, 7.87), turned to 180 degrees
- moved R4 63.7 mm to (55.6, 6.22), turned to 180 degrees
- moved C12 61.2 mm to (48.9, 16.0), turned to 270 degrees
- moved U19 54.4 mm to (-26.4, 8.64), turned to 270 degrees
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- renumbered J6 to J2, J7 to J3, J8 to J4, J9 to J5, U28 to U10, U31 to U9
Connections:
- net !FAULT1: now also U1.9, U2.9, U8.24; no longer U26.24, U5.9, U6.9
- net !FAULT2: now also U1.3, U2.13, U8.1; no longer U26.1, U5.13, U6.3
- net !FAULT3: now also U1.5, U2.10, U8.2; no longer U26.2, U5.10, U6.5
- net !FAULT4: now also U1.1, U2.1, U8.3; no longer U26.3, U5.1, U6.1
- net !I2C_OB_EN: now also U1.10, U18.1, U19.1, U20.1, U21.1; no longer U12.1, U13.1, U14.1, U15.1, U6.10
- net 3V3: now also C4.1, C6.1, C8.1, Q6.2, Q8.2, R12.2, R13.2, R17.2, R18.2, R2.2, U1.13, U1.14, U11.5, U13.1, U13.8, U14.7, U15.7, U16.7, U18.5, U19.5, U2.16, U2.5, U20.5, U21.5, U3.3, U7.4, U8.12, U8.8; no longer C11.1, C12.1, C13.1, Q1.2, Q3.2, R16.2, R22.2, R5.2, R6.2, R9.2, U11.4, U13.5, U14.5, U15.5, U16.1, U16.8, U18.7, U19.7, U20.7, U26.12, U26.8, U29.5, U30.5, U5.16, U5.5, U6.13, U7.14, U8.3
- net 3V3_SENSE: now also C2.1, R10.2, U3.1, U5.4; no longer C8.1, R8.2, U3.4, U8.1
- net DATA1_EN: now also U18.2, U8.19; no longer U12.2, U26.19
- net DATA1_EN_LOCAL: now also U14.3, U18.4; no longer U12.4, U17.3
- net DATA2_EN: now also U19.2, U8.20; no longer U13.2, U26.20
- net DATA2_EN_LOCAL: now also U15.3, U19.4; no longer U13.4, U18.3
- net DATA3_EN: now also U20.2, U8.21; no longer U14.2, U26.21
- net DATA3_EN_LOCAL: now also U16.3, U20.4; no longer U14.4, U19.3
- net DATA4_EN: now also U21.2, U8.22; no longer U15.2, U26.22
- net DATA4_EN_LOCAL: now also U17.3, U21.4; no longer U15.4, U20.3
- net EN1: now also U2.6, U6.12, U8.15; no longer U26.15, U5.6, U7.12
- net EN2: now also U2.4, U6.1, U8.16; no longer U26.16, U5.4, U7.1
- net EN3: now also U2.12, U6.9, U8.17; no longer U26.17, U5.12, U7.9
- net EN4: now also U2.14, U6.4, U8.18; no longer U26.18, U5.14, U7.4
- net FAULT1: now also U1.8, U6.13; no longer U6.8, U7.13
- net FAULT2: now also U1.4, U6.2; no longer U6.4, U7.2
- net FAULT3: now also U1.6, U6.10; no longer U6.6, U7.10
- net FAULT4: now also U1.2, U6.5; no longer U6.2, U7.5
- net GND: now also Q1.2, Q3.2, R16.1, R9.1, U1.7, U12.2, U12.6, U13.4, U14.2, U14.EP, U15.2, U15.EP, U16.2, U16.EP, U18.3, U19.3, U2.8, U20.3, U21.3, U3.2, U3.EP, U5.11, U7.2, U7.5, U8.23; no longer Q6.2, Q8.2, R13.1, R21.1, U11.5, U12.3, U13.3, U14.3, U15.3, U16.4, U18.2, U18.EP, U19.2, U19.EP, U20.2, U20.EP, U26.23, U26.EP, U29.2, U3.11, U30.2, U30.6, U5.8, U7.7, U8.2
- net I2C_OB_EN: now also R12.1, U1.11, U13.5; no longer R16.1, U16.5, U6.11
- net INTB: now also U8.13; no longer U26.13
- net LATCH1: now also U2.7, U5.1; no longer U3.1, U5.7
- net LATCH2: now also U2.3, U5.7; no longer U3.7, U5.3
- net LATCH3: now also U2.11, U5.8; no longer U3.8, U5.11
- net LATCH4: now also U2.15, U5.14; no longer U3.14, U5.15
- net MOS_CTRL1: now also Q1.1, U6.11; no longer Q2.1, U7.11
- net MOS_CTRL2: now also Q2.1, U6.3; no longer Q4.1, U7.3
- net MOS_CTRL3: now also Q3.1, U6.8; no longer Q6.1, U7.8
- net MOS_CTRL4: now also Q4.1, U6.6; no longer Q8.1, U7.6
- net MUX_SEL2: now also U11.4; no longer U29.4
- net N$1: now also Q2.3, Q6.1, R2.1; no longer Q3.1, Q4.3, R9.1
- net N$14: now also R13.1, R14.2, U8.11; no longer R21.2, R22.1, U26.11
- net N$2: now also Q1.3, Q5.1, R1.1; no longer Q1.1, Q2.3, R6.1
- net N$3: now also Q3.3, Q7.1, R3.1; no longer Q5.1, Q6.3, R11.1
- net N$38: now also U11.1; no longer U29.1
- net N$4: now also Q4.3, Q8.1, R4.1; no longer Q7.1, Q8.3, R1.1
- net N$6: now also R16.2, U11.3; no longer R14.2, U29.3
- net PORT1_SCL: now also R23.1, U14.5; no longer R20.1, U17.5
- net PORT1_SDA: now also U14.4; no longer U17.4
- net PORT2_SCL: now also U15.5; no longer U18.5
- net PORT2_SDA: now also R20.1, U15.4; no longer R23.1, U18.4
- net PORT3_SCL: now also R25.1, U16.5; no longer R18.1, U19.5
- net PORT3_SDA: now also R21.1, U16.4; no longer R17.1, U19.4
- net PORT4_SCL: now also U17.5; no longer U20.5
- net PORT4_SDA: now also R22.1, U17.4; no longer R25.1, U20.4
- net POS_DETECT: now also R11.1, U8.4; no longer R5.1, U26.4
- net SCL: now also R18.1, U13.3, U14.8, U15.8, U16.8; no longer R4.1, U16.3, U18.8, U19.8, U20.8
- net SCL_OB: now also U12.3, U13.6, U7.1, U8.9; no longer U11.1, U16.6, U26.9, U30.3
- net SDA: now also R17.1, U13.2, U14.1, U15.1, U16.1; no longer R3.1, U16.2, U18.1, U19.1, U20.1
- net SDA_OB: now also U12.4, U13.7, U7.3, U8.10; no longer U11.3, U16.7, U26.10, U30.4
- net SENSE1: now also U5.2; no longer U3.2
- net SENSE1+: now also Q5.3, R5.1; no longer Q1.3, R7.1
- net SENSE2: now also U5.6; no longer U3.6
- net SENSE2+: now also Q6.3, R6.1; no longer Q3.3, R10.1
- net SENSE3: now also U5.9; no longer U3.9
- net SENSE3+: now also Q7.3, R7.1; no longer Q5.3, R12.1
- net SENSE4: now also U5.13; no longer U3.13
- net SENSE4+: now also Q8.3, R8.1; no longer Q7.3, R2.1
- net SENSE_EN: now also R9.2, U3.4, U8.5; no longer R13.2, U26.5, U8.4
- net SWITCHED_SENSE: now also U11.6, U12.1; no longer U29.6, U30.1
- net VPORT1_OUT: now also C13.1, R23.2, R5.2, U14.6; no longer C2.1, R20.2, R7.2, U17.6
- net VPORT2_OUT: now also C10.1, R20.2, R6.2, U15.6; no longer C4.1, R10.2, R23.2, U18.6
- net VPORT3_OUT: now also C11.1, R21.2, R25.2, R7.2, U16.6; no longer C6.1, R12.2, R17.2, R18.2, U19.6
- net VPORT4_OUT: now also C12.1, R22.2, R8.2, U17.6; no longer C10.1, R2.2, R25.2, U20.6
- net VREF: now also R10.1, U5.10, U5.12, U5.3, U5.5; no longer R8.1, U3.10, U3.12, U3.3, U3.5
Other:
- board text added: "Port1"
- board text added: "Port2"
- board text added: "Port3"
- board text added: "Port4"
- board text added: "Talon - I2C v0.0 Bobby Schulz"

Commit message: Layout, gerbers and BoM for v0.0 - submitted to fab
Parts:
- added TP1, TP2, TP3, TP4, TP5, TP6: TESTPOINTRCU, bschulz:TESTPOINT_0603
- R13: value (none) -> 110k
- R14: value (none) -> 49.9k
- R15, R16: value (none) -> 10k
Connections:
- net GND: now also TP1.1
- net INTB: now also TP6.1
- net SCL: now also TP3.1
- net SCL_OB: now also TP5.1
- net SDA: now also TP2.1
- net SDA_OB: now also TP4.1
Routing:
- net SCL: track 145.3 -> 151.0 mm
- net SDA: track 143.3 -> 145.9 mm
- net INTB: track 37.2 -> 39.6 mm
- net SDA_OB: track 34.3 -> 35.7 mm
- net GND: track 372.8 -> 374.1 mm
- net SCL_OB: track 29.5 -> 30.4 mm
- net VPORT4_OUT: track 189.3 -> 189.9 mm
- net SENSE4+: track 102.7 -> 103.3 mm
- net VPORT3_OUT: track 110.7 -> 111.3 mm
- net SENSE3+: track 70.2 -> 70.8 mm
Other:
- board text added: "GND"
- board text added: "INTB"
- board text added: "SCL"
- board text added: "SCL_OB"
- board text added: "SDA"
- board text added: "SDA_OB"
- board text added: "SN"
