File: Hardware/Talon_I2C.sch (EAGLE design)
At the start: 88 parts, among them J1 CONN_TALON_REMOTE, J2 CONN_SDI-12_LOGGERM8_TE_BOARD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, J3 CONN_SDI-12_LOGGERM8_TE_BOARD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, J4 CONN_SDI-12_LOGGERM8_TE_BOARD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, J5 CONN_APOGEE_LOGGER, Q1 AO3419, Q2 2N7002, Q3 AO3419, Q4 2N7002, Q5 AO3419, Q6 2N7002, Q7 AO3419, Q8 2N7002, U1 SN74LVC1G00SC70, U10 SN74LVC1G3157SC70, U11 SN74LVC1G3157SC70, U12 SN74LVC1G3157SC70, U13 SN74LVC1G3157SC70, U14 LM2621, U15 MCP3221, U16 LMR62014SOT23, U17 TXS0102DCU, U18 FDC6330L, U2 SN74LVC2G241DCU, U26 MCP23018QFN, U28 74HC4852, U29 SN74AUP1T157DCK, U3 MAX9034TSSOP, U30 MCP3421A3, U31 PCA9536DFN, U4 INA4180A2, U5 CD4044, U6 SN74HC04, U7 SN74AC08, U8 SIP32431TDFN, U9 SN74LVC1G17DCK

Commit message: Copper layout done
Parts:
- removed C14: 10uF, bschulz_passives:C-EU10UFC0805
- removed C15: 220pF, bschulz_passives:C-EU220PFC0603
- removed C16: 0.1uF, bschulz_passives:C-EU0.1UFC0603
- removed D2: CDBA3100, bschulz:DIODE_SCHOTTKYDO-214AC
- removed D4: (no value), bschulz:DIODE_SCHOTTKYSOD-123
- removed J2, J3, J4: CONN_SDI-12_LOGGERM8_TE_BOARDLOCK, GEMS_Plugs:CONN_SDI-12_LOGGERM8_TE_BOARDLOCK
- removed J5: CONN_APOGEE_LOGGER, GEMS_Plugs:CONN_APOGEE_LOGGER
- removed L1: 6.8uH, bschulz:INDUCTOR_MAIA_4.1X4.1
- removed L3: 10uH, bschulz:INDUCTOR_1008
- removed R27, R28: 100k, bschulz_passives:R-EU_100KR0603
- removed R31: 40.2k, bschulz_passives:R-EU_115KR0603
- removed R32: 13.3k, bschulz_passives:R-EU_13.3KR0603
- removed U1: SN74LVC1G00SC70, bschulz:SN74LVC1G00SC70
- removed U10: SN74LVC1G3157SC70, bschulz:SN74LVC1G3157SC70
- removed U2: SN74LVC2G241DCU, bschulz:SN74LVC2G241DCU
- removed U9: SN74LVC1G17DCK, bschulz:SN74LVC1G17DCK
- added J6, J7, J8, J9: CONN_I2C_LOGGER, GEMS_Plugs:CONN_I2C_LOGGER
- added U19, U20: PCA9617WSON, bschulz:PCA9617WSON
- C1, C10, C12, C3, C6, C8: device bschulz_passives:C-EU0.1UFC0603 -> bschulz_passives:C-EU0.1UFC0402
- C11: value 4.7uF -> 0.1uF; device bschulz_passives:C-EU4.7UFC0805 -> bschulz_passives:C-EU0.1UFC0402
- C2: value 22uF -> 0.1uF; device bschulz_passives:C-EU22UFC0805 -> bschulz_passives:C-EU0.1UFC0402
- C4: value (none) -> 0.1uF; device bschulz_passives:C-EUC0603 -> bschulz_passives:C-EU0.1UFC0402
- C5: value 68uF -> 0.1uF; device bschulz_passives:CTANT_EU2917 -> bschulz_passives:C-EU0.1UFC0402
- C9: value 10uF -> 0.1uF; device bschulz_passives:C-EU10UFC0805 -> bschulz_passives:C-EU0.1UFC0402
- R1, R11, R3, R4, R6, R8, R9: device bschulz_passives:R-EU_10KR0603 -> bschulz_passives:R-EU_10KR0402
- R13: device bschulz_passives:R-EU_100KR0603 -> bschulz_passives:R-EU_100KR0402
- R14, R15: device bschulz_passives:R-EU_R0603 -> bschulz_passives:R-EU_R0402
- R16: value (none) -> 100k; device bschulz_passives:R-EU_R0603 -> bschulz_passives:R-EU_100KR0402
- R17, R18, R19, R20, R23: device bschulz_passives:R-EU_R0603 -> bschulz_passives:R-EU_10KR0402
- R24: value 470k -> (none); device bschulz_passives:R-EU_470KR0603 -> bschulz_passives:R-EU_10KR0402
- R25: value 115k -> (none); device bschulz_passives:R-EU_115KR0603 -> bschulz_passives:R-EU_10KR0402
- R26: value 13.3k -> (none); device bschulz_passives:R-EU_13.3KR0603 -> bschulz_passives:R-EU_10KR0402
- R5: device bschulz_passives:R-EU_1MR0603 -> bschulz_passives:R-EU_1MR0402
- U11: value SN74LVC1G3157SC70 -> 24AA02SOT23; device bschulz:SN74LVC1G3157SC70 -> bschulz:24AA02SOT23
- U12, U13: value SN74LVC1G3157SC70 -> SN74AUP1G08DCK; device bschulz:SN74LVC1G3157SC70 -> bschulz:SN74AUP1G08DCK
- U14: value LM2621 -> SN74AUP1G08DCK; device bschulz:LM2621 -> bschulz:SN74AUP1G08DCK
- U15: value MCP3221 -> SN74AUP1G08DCK; device bschulz:MCP3221 -> bschulz:SN74AUP1G08DCK
- U16: value LMR62014SOT23 -> FXMAR2102UMLP; device bschulz:LMR62014SOT23 -> bschulz:FXMAR2102UMLP
- U17: value TXS0102DCU -> PCA9617WSON; device bschulz:TXS0102DCU -> bschulz:PCA9617WSON
- U18: value FDC6330L -> PCA9617WSON; device bschulz:FDC6330L -> bschulz:PCA9617WSON
Connections:
- removed net !RX: U2.1Y, U9.A
- removed net 12V: C4.1, C5.+, D2.C, Q1.S, Q3.S, Q5.S, Q7.S, R1.2, R11.2, R25.2, R27.2, R6.2, R9.2, U18.VIN
- removed net 5V: C14.1, C15.1, C16.1, C6.1, C9.1, D4.C, R31.2, U10.VCC, U11.VCC, U12.VCC, U13.VCC, U15.VDD, U17.VB, U2.VCC
- removed net DATA: U10.B2, U11.B2, U12.B2, U13.B2, U2.1A, U2.2Y
- removed net DATA_EN1: U10.S, U26.GPA4
- removed net DATA_EN2: U11.S, U26.GPA5
- removed net DATA_EN3: U12.S, U26.GPA6
- removed net DATA_EN4: R28.2, U13.S, U18.EN, U26.GPA7
- removed net DATA_OUT1: J2.DATA, U10.A
- removed net DATA_OUT2: J3.DATA, U11.A
- removed net DATA_OUT3: J4.DATA, U12.A
- removed net DATA_OUT4: J5.3, U13.A
- removed net DATA_SENSE4: U13.B1, U15.VIN
- removed net DIR: U2.1!OE, U2.2OE, U26.GPB7
- removed net FOUT: U1.A, U26.GPB6
- removed net N$10: C15.2, R31.1, R32.2, U16.FB
- removed net N$11: R27.1, U18.R1,C1
- removed net N$18: U28.2Z, U29.B
- removed net N$7: C3.2, R24.1, U14.FREQ
- removed net N$8: D2.A, L1.2, U14.SW
- removed net N$9: C4.2, R25.1, R26.2, U14.FB
- removed net RX: J1.RX, U9.Y
- removed net SCL_HV: U15.SCL, U17.B2
- removed net SDA_HV: U15.SDA, U17.B1
- removed net SW1: D4.A, L3.2, U16.SW
- removed net TX: J1.TX, U1.B
- removed net VHEATER: J5.5, U18.VOUT
- removed net VPORT1_OUT_SENSE: R14.2, R15.2, U28.2Y0
- removed net VPORT2_OUT_SENSE: R16.2, R17.2, U28.2Y1
- removed net VPORT3_OUT_SENSE: R18.2, R19.2, U28.2Y2
- removed net VPORT4_OUT_SENSE: R20.2, R23.2, U28.2Y3
- new net !I2C_OB_EN: U12.A, U13.A, U14.A, U15.A, U6.Y5
- new net DATA1_EN: U12.B, U26.GPA4
- new net DATA1_EN_LOCAL: U12.Y, U17.EN
- new net DATA2_EN: U13.B, U26.GPA5
- new net DATA2_EN_LOCAL: U13.Y, U18.EN
- new net DATA3_EN: U14.B, U26.GPA6
- new net DATA3_EN_LOCAL: U14.Y, U19.EN
- new net DATA4_EN: U15.B, U26.GPA7
- new net DATA4_EN_LOCAL: U15.Y, U20.EN
- new net I2C_OB_EN: J1.RX, R16.1, U16.EN, U6.A5
- new net INTB: J1.TX, U26.INTB
- new net N$6: R14.2, R15.1, U29.B
- new net PORT1_SCL: J6.SCL, R20.1, U17.SCL_B
- new net PORT1_SDA: J6.SDA, R19.1, U17.SDA_B
- new net PORT2_SCL: J7.SCL, R24.1, U18.SCL_B
- new net PORT2_SDA: J7.SDA, R23.1, U18.SDA_B
- new net PORT3_SCL: J8.SCL, R18.1, U19.SCL_B
- new net PORT3_SDA: J8.SDA, R17.1, U19.SDA_B
- new net PORT4_SCL: J9.SCL, R26.1, U20.SCL_B
- new net PORT4_SDA: J9.SDA, R25.1, U20.SDA_B
- new net SCL_OB: U11.SCL, U16.B2, U26.SCL, U30.SCL, U31.SCL
- new net SDA_OB: U11.SDA, U16.B1, U26.SDA, U30.SDA, U31.SDA
- net 3V3: now also C5.1, C9.1, Q1.S, Q3.S, Q5.S, Q7.S, R1.2, R11.2, R16.2, R6.2, R9.2, U11.VCC, U12.VCC, U13.VCC, U14.VCC, U15.VCC, U16.VA, U16.VB, U17.VCCA, U18.VCCA, U19.VCCA, U20.VCCA; no longer C10.1, C2.1, L1.1, L3.1, R24.2, U1.VCC, U14.BOOT, U14.EN, U14.VDD, U16.!SHDN, U16.VIN, U17.EN, U17.VA, U6.A5, U9.VCC
- net GND: now also C3.2, C4.2, C5.2, J6.GND, J7.GND, J8.GND, J9.GND, R14.1, U11.WP, U14.GND, U15.GND, U18.GND, U19.GND, U20.GND; no longer C14.2, C16.2, C5.-, J2.GND, J3.GND, J4.GND, J5.1, J5.6, R15.1, R17.1, R19.1, R23.1, R26.1, R28.1, R32.1, U1.GND, U10.GND, U14.PGND, U14.SGND, U15.VSS, U18.R2, U2.GND, U9.GND
- net N$5: now also R15.2, U28.2Z; no longer U1.Y, U2.2A
- net SCL: now also U16.A2, U17.SCL_A, U18.SCL_A, U19.SCL_A, U20.SCL_A; no longer U17.A2, U26.SCL, U30.SCL, U31.SCL
- net SDA: now also U16.A1, U17.SDA_A, U18.SDA_A, U19.SDA_A, U20.SDA_A; no longer U17.A1, U26.SDA, U30.SDA, U31.SDA
- net VPORT1_OUT: now also C2.1, J6.3V3, R19.2, R20.2, U17.VCCB, U28.2Y0; no longer J2.12V, R14.1
- net VPORT2_OUT: now also C4.1, J7.3V3, R23.2, R24.2, U18.VCCB, U28.2Y1; no longer J3.12V, R16.1
- net VPORT3_OUT: now also C6.1, J8.3V3, R17.2, R18.2, U19.VCCB, U28.2Y2; no longer J4.12V, R18.1
- net VPORT4_OUT: now also C10.1, J9.3V3, R25.2, R26.2, U20.VCCB, U28.2Y3; no longer J5.2, R20.1
Other:
- note removed: "Change this to a dedicated pin in future?"
- note removed: "Pull down to ensure system does not apply 12V to heater lines until tested"
- note removed: "REPLACE! SN74LVC1G14"
- note removed: "TVS DIODES"

Commit message: Generated gerbers for v0.0
Ready for final review
Parts:
- removed J6, J7, J8, J9: CONN_I2C_LOGGER, GEMS_Plugs:CONN_I2C_LOGGER
- removed U26: MCP23018QFN, bschulz:MCP23018QFN
- removed U28: 74HC4852, bschulz:74HC4852
- removed U29: SN74AUP1T157DCK, bschulz:SN74AUP1T157DCK
- removed U30: MCP3421A3, bschulz:MCP3421A3
- removed U31: PCA9536DFN, bschulz:PCA9536DFN
- added J2, J3, J4, J5: CONN_I2C_LOGGER, GEMS_Plugs:CONN_I2C_LOGGER
- added U1: SN74HC04, bschulz:SN74HC04
- added U10: 74HC4852, bschulz:74HC4852
- added U2: CD4044, bschulz:CD4044
- added U21: SN74AUP1G08DCK, bschulz:SN74AUP1G08DCK
- added U9: PCA9536DFN, bschulz:PCA9536DFN
- C1: value 0.1uF -> 1uF; device bschulz_passives:C-EU0.1UFC0402 -> bschulz_passives:C-EU1UFC0603
- C13: value 10uF -> 0.1uF; device bschulz_passives:C-EU10UFC0805 -> bschulz_passives:C-EU0.1UFC0402
- C4: value 0.1uF -> 10uF; device bschulz_passives:C-EU0.1UFC0402 -> bschulz_passives:C-EU10UFC0805
- C7: value 1uF -> 0.1uF; device bschulz_passives:C-EU1UFC0603 -> bschulz_passives:C-EU0.1UFC0402
- Q1, Q3: value AO3419 -> 2N7002; device bschulz:MOSFET-PCH-AO3419 -> bschulz:MOSFET-NCH-2N7002P
- Q6, Q8: value 2N7002 -> AO3419; device bschulz:MOSFET-NCH-2N7002P -> bschulz:MOSFET-PCH-AO3419
- R10, R2: value 82m -> 10k; device bschulz_passives:R-EU_R0603 -> bschulz_passives:R-EU_10KR0402
- R11: value 10k -> 1M; device bschulz_passives:R-EU_10KR0402 -> bschulz_passives:R-EU_1MR0402
- R12: value 82m -> 100k; device bschulz_passives:R-EU_R0603 -> bschulz_passives:R-EU_100KR0402
- R13: value 100k -> (none); device bschulz_passives:R-EU_100KR0402 -> bschulz_passives:R-EU_R0603
- R14: device bschulz_passives:R-EU_R0402 -> bschulz_passives:R-EU_R0603
- R16: value 100k -> (none); device bschulz_passives:R-EU_100KR0402 -> bschulz_passives:R-EU_R0402
- R17, R18, R19, R20, R23, R24, R25, R26: value (none) -> 10k
- R21, R22: value (none) -> 10k; device bschulz_passives:R-EU_R0603 -> bschulz_passives:R-EU_10KR0402
- R5: value 1M -> 82m; device bschulz_passives:R-EU_1MR0402 -> bschulz_passives:R-EU_R0603
- R6, R8: value 10k -> 82m; device bschulz_passives:R-EU_10KR0402 -> bschulz_passives:R-EU_R0603
- R9: value 10k -> 100k; device bschulz_passives:R-EU_10KR0402 -> bschulz_passives:R-EU_100KR0402
- U11: value 24AA02SOT23 -> SN74AUP1T157DCK; device bschulz:24AA02SOT23 -> bschulz:SN74AUP1T157DCK
- U12: value SN74AUP1G08DCK -> MCP3421A3; device bschulz:SN74AUP1G08DCK -> bschulz:MCP3421A3
- U13: value SN74AUP1G08DCK -> FXMAR2102UMLP; device bschulz:SN74AUP1G08DCK -> bschulz:FXMAR2102UMLP
- U14, U15: value SN74AUP1G08DCK -> PCA9617WSON; device bschulz:SN74AUP1G08DCK -> bschulz:PCA9617WSON
- U16: value FXMAR2102UMLP -> PCA9617WSON; device bschulz:FXMAR2102UMLP -> bschulz:PCA9617WSON
- U18, U19, U20: value PCA9617WSON -> SN74AUP1G08DCK; device bschulz:PCA9617WSON -> bschulz:SN74AUP1G08DCK
- U3: value MAX9034TSSOP -> SIP32431TDFN; device bschulz:MAX9034TSSOP -> bschulz:SIP32431TDFN
- U5: value CD4044 -> MAX9034TSSOP; device bschulz:CD4044 -> bschulz:MAX9034TSSOP
- U6: value SN74HC04 -> SN74AC08; device bschulz:SN74HC04 -> bschulz:SN74AC08
- U7: value SN74AC08 -> 24AA02SOT23; device bschulz:SN74AC08 -> bschulz:24AA02SOT23
- U8: value SIP32431TDFN -> MCP23018QFN; device bschulz:SIP32431TDFN -> bschulz:MCP23018QFN
Connections:
- net !FAULT1: now also U1.A4, U2.Q2, U8.GPB0; no longer U26.GPB0, U5.Q2, U6.A4
- net !FAULT2: now also U1.A2, U2.Q1, U8.GPB1; no longer U26.GPB1, U5.Q1, U6.A2
- net !FAULT3: now also U1.A3, U2.Q3, U8.GPB2; no longer U26.GPB2, U5.Q3, U6.A3
- net !FAULT4: now also U1.A1, U2.Q4, U8.GPB3; no longer U26.GPB3, U5.Q4, U6.A1
- net !I2C_OB_EN: now also U1.Y5, U18.A, U19.A, U20.A, U21.A; no longer U12.A, U13.A, U14.A, U15.A, U6.Y5
- net 3V3: now also C4.1, C6.1, C8.1, Q6.S, Q8.S, R12.2, R13.2, R17.2, R18.2, R2.2, U1.A6, U1.VCC, U10.VCC, U12.VDD, U13.VA, U13.VB, U14.VCCA, U15.VCCA, U16.VCCA, U18.VCC, U19.VCC, U2.EN, U2.VCC, U20.VCC, U21.VCC, U3.VIN, U8.!RESET, U8.VDD, U9.VCC; no longer C11.1, C12.1, C13.1, Q1.S, Q3.S, R16.2, R22.2, R5.2, R6.2, R9.2, U12.VCC, U13.VCC, U14.VCC, U15.VCC, U16.VA, U16.VB, U18.VCCA, U19.VCCA, U20.VCCA, U26.!RESET, U26.VDD, U28.VCC, U29.VCC, U30.VDD, U31.VCC, U5.EN, U5.VCC, U6.A6, U8.VIN
- net 3V3_SENSE: now also C2.1, R10.2, U3.VOUT, U5.VDD; no longer C8.1, R8.2, U3.VDD, U8.VOUT
- net DATA1_EN: now also U18.B, U8.GPA4; no longer U12.B, U26.GPA4
- net DATA1_EN_LOCAL: now also U14.EN, U18.Y; no longer U12.Y, U17.EN
- net DATA2_EN: now also U19.B, U8.GPA5; no longer U13.B, U26.GPA5
- net DATA2_EN_LOCAL: now also U15.EN, U19.Y; no longer U13.Y, U18.EN
- net DATA3_EN: now also U20.B, U8.GPA6; no longer U14.B, U26.GPA6
- net DATA3_EN_LOCAL: now also U16.EN, U20.Y; no longer U14.Y, U19.EN
- net DATA4_EN: now also U21.B, U8.GPA7; no longer U15.B, U26.GPA7
- net DATA4_EN_LOCAL: now also U17.EN, U21.Y; no longer U15.Y, U20.EN
- net EN1: now also U2.R2, U6.A4, U8.GPA0; no longer U26.GPA0, U5.R2, U7.A4
- net EN2: now also U2.R1, U6.A1, U8.GPA1; no longer U26.GPA1, U5.R1, U7.A1
- net EN3: now also U2.R3, U6.A3, U8.GPA2; no longer U26.GPA2, U5.R3, U7.A3
- net EN4: now also U2.R4, U6.A2, U8.GPA3; no longer U26.GPA3, U5.R4, U7.A2
- net FAULT1: now also U1.Y4, U6.B4; no longer U6.Y4, U7.B4
- net FAULT2: now also U1.Y2, U6.B1; no longer U6.Y2, U7.B1
- net FAULT3: now also U1.Y3, U6.B3; no longer U6.Y3, U7.B3
- net FAULT4: now also U1.Y1, U6.B2; no longer U6.Y1, U7.B2
- net GND: now also J2.GND, J3.GND, J4.GND, J5.GND, Q1.S, Q3.S, R16.1, R9.1, U1.GND, U10.GND, U12.VIN-, U12.VSS, U2.GND, U21.GND, U7.WP, U8.VSS, U9.GND; no longer J6.GND, J7.GND, J8.GND, J9.GND, Q6.S, Q8.S, R13.1, R21.1, U11.WP, U12.GND, U26.VSS, U28.GND, U29.GND, U30.VIN-, U30.VSS, U31.GND, U8.GND
- net I2C_OB_EN: now also R12.1, U1.A5, U13.EN; no longer R16.1, U16.EN, U6.A5
- net INTB: now also U8.INTB; no longer U26.INTB
- net LATCH1: now also U2.S2, U5.OUTA; no longer U3.OUTA, U5.S2
- net LATCH2: now also U2.S1, U5.OUTB; no longer U3.OUTB, U5.S1
- net LATCH3: now also U2.S3, U5.OUTC; no longer U3.OUTC, U5.S3
- net LATCH4: now also U2.S4, U5.OUTD; no longer U3.OUTD, U5.S4
- net MOS_CTRL1: now also Q1.G, U6.Y4; no longer Q2.G, U7.Y4
- net MOS_CTRL2: now also Q2.G, U6.Y1; no longer Q4.G, U7.Y1
- net MOS_CTRL3: now also Q3.G, U6.Y3; no longer Q6.G, U7.Y3
- net MOS_CTRL4: now also Q4.G, U6.Y2; no longer Q8.G, U7.Y2
- net MUX_EN: now also U10.!E, U9.P3; no longer U28.!E, U31.P3
- net MUX_SEL0: now also U10.S0, U9.P0; no longer U28.S0, U31.P0
- net MUX_SEL1: now also U10.S1, U9.P1; no longer U28.S1, U31.P1
- net MUX_SEL2: now also U11.C, U9.P2; no longer U29.C, U31.P2
- net N$1: now also Q2.D, Q6.G, R2.1; no longer Q3.G, Q4.D, R9.1
- net N$14: now also R13.1, R14.2, U8.ADDR; no longer R21.2, R22.1, U26.ADDR
- net N$2: now also Q1.D, Q5.G, R1.1; no longer Q1.G, Q2.D, R6.1
- net N$3: now also Q3.D, Q7.G, R3.1; no longer Q5.G, Q6.D, R11.1
- net N$38: now also U10.1Z, U11.A; no longer U28.1Z, U29.A
- net N$4: now also Q4.D, Q8.G, R4.1; no longer Q7.G, Q8.D, R1.1
- net N$5: now also U10.2Z; no longer U28.2Z
- net N$6: now also R16.2, U11.B; no longer R14.2, U29.B
- net PORT1_SCL: now also J2.SCL, R23.1, U14.SCL_B; no longer J6.SCL, R20.1, U17.SCL_B
- net PORT1_SDA: now also J2.SDA, U14.SDA_B; no longer J6.SDA, U17.SDA_B
- net PORT2_SCL: now also J3.SCL, U15.SCL_B; no longer J7.SCL, U18.SCL_B
- net PORT2_SDA: now also J3.SDA, R20.1, U15.SDA_B; no longer J7.SDA, R23.1, U18.SDA_B
- net PORT3_SCL: now also J4.SCL, R25.1, U16.SCL_B; no longer J8.SCL, R18.1, U19.SCL_B
- net PORT3_SDA: now also J4.SDA, R21.1, U16.SDA_B; no longer J8.SDA, R17.1, U19.SDA_B
- net PORT4_SCL: now also J5.SCL, U17.SCL_B; no longer J9.SCL, U20.SCL_B
- net PORT4_SDA: now also J5.SDA, R22.1, U17.SDA_B; no longer J9.SDA, R25.1, U20.SDA_B
- net POS_DETECT: now also R11.1, U8.GPB4; no longer R5.1, U26.GPB4
- net SCL: now also R18.1, U13.A2, U14.SCL_A, U15.SCL_A, U16.SCL_A; no longer R4.1, U16.A2, U18.SCL_A, U19.SCL_A, U20.SCL_A
- net SCL_OB: now also U12.SCL, U13.B2, U7.SCL, U8.SCL, U9.SCL; no longer U11.SCL, U16.B2, U26.SCL, U30.SCL, U31.SCL
- net SDA: now also R17.1, U13.A1, U14.SDA_A, U15.SDA_A, U16.SDA_A; no longer R3.1, U16.A1, U18.SDA_A, U19.SDA_A, U20.SDA_A
- net SDA_OB: now also U12.SDA, U13.B1, U7.SDA, U8.SDA, U9.SDA; no longer U11.SDA, U16.B1, U26.SDA, U30.SDA, U31.SDA
- net SENSE1: now also U10.1Y0, U5.INA-; no longer U28.1Y0, U3.INA-
- net SENSE1+: now also Q5.D, R5.1; no longer Q1.D, R7.1
- net SENSE2: now also U10.1Y1, U5.INB-; no longer U28.1Y1, U3.INB-
- net SENSE2+: now also Q6.D, R6.1; no longer Q3.D, R10.1
- net SENSE3: now also U10.1Y2, U5.INC-; no longer U28.1Y2, U3.INC-
- net SENSE3+: now also Q7.D, R7.1; no longer Q5.D, R12.1
- net SENSE4: now also U10.1Y3, U5.IND-; no longer U28.1Y3, U3.IND-
- net SENSE4+: now also Q8.D, R8.1; no longer Q7.D, R2.1
- net SENSE_EN: now also R9.2, U3.EN, U8.GPB5; no longer R13.2, U26.GPB5, U8.EN
- net SWITCHED_SENSE: now also U11.Y, U12.VIN+; no longer U29.Y, U30.VIN+
- net VPORT1_OUT: now also C13.1, J2.3V3, R23.2, R5.2, U10.2Y0, U14.VCCB; no longer C2.1, J6.3V3, R20.2, R7.2, U17.VCCB, U28.2Y0
- net VPORT2_OUT: now also C10.1, J3.3V3, R20.2, R6.2, U10.2Y1, U15.VCCB; no longer C4.1, J7.3V3, R10.2, R23.2, U18.VCCB, U28.2Y1
- net VPORT3_OUT: now also C11.1, J4.3V3, R21.2, R25.2, R7.2, U10.2Y2, U16.VCCB; no longer C6.1, J8.3V3, R12.2, R17.2, R18.2, U19.VCCB, U28.2Y2
- net VPORT4_OUT: now also C12.1, J5.3V3, R22.2, R8.2, U10.2Y3, U17.VCCB; no longer C10.1, J9.3V3, R2.2, R25.2, U20.VCCB, U28.2Y3
- net VREF: now also R10.1, U5.INA+, U5.INB+, U5.INC+, U5.IND+; no longer R8.1, U3.INA+, U3.INB+, U3.INC+, U3.IND+

Commit message: Layout, gerbers and BoM for v0.0 - submitted to fab
Parts:
- added TP1, TP2, TP3, TP4, TP5, TP6: TESTPOINTRCU, bschulz:TESTPOINTRCU
- R13: value (none) -> 110k; device bschulz_passives:R-EU_R0603 -> bschulz_passives:R-EU_110KR0603
- R14: value (none) -> 49.9k; device bschulz_passives:R-EU_R0603 -> bschulz_passives:R-EU_49.9KR0603
- R15, R16: value (none) -> 10k; device bschulz_passives:R-EU_R0402 -> bschulz_passives:R-EU_10KR0402
- R5, R6, R7, R8: device bschulz_passives:R-EU_R0603 -> bschulz_passives:R-EU_0.082R0603
Connections:
- net GND: now also TP1.P$1
- net INTB: now also TP6.P$1
- net SCL: now also TP3.P$1
- net SCL_OB: now also TP5.P$1
- net SDA: now also TP2.P$1
- net SDA_OB: now also TP4.P$1
Other:
- note added: "ADR: 0x22"
- note added: "Fix!"
Changed lines of the file:
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@@
 <part name="U6" library="bschulz" deviceset="SN74AC08" device=""/>
 <part name="GND12" library="supply1" library_urn="urn:adsk.eagle:library:371" deviceset="GND" device=""/>
-<part name="R5" library="bschulz_passives" deviceset="R-EU_" device="R0603" value="82m"/>
+<part name="R5" library="bschulz_passives" deviceset="R-EU_" device="R0603" technology="0.082" value="82m"/>
 <part name="GND13" library="supply1" library_urn="urn:adsk.eagle:library:371" deviceset="GND" device=""/>
 <part name="GND14" library="supply1" library_urn="urn:adsk.eagle:library:371" deviceset="GND" device=""/>
@@
 <part name="R2" library="bschulz_passives" deviceset="R-EU_" device="R0402" technology="10K" value="10k"/>
 <part name="GND19" library="supply1" library_urn="urn:adsk.eagle:library:371" deviceset="GND" device=""/>
-<part name="R6" library="bschulz_passives" deviceset="R-EU_" device="R0603" value="82m"/>
+<part name="R6" library="bschulz_passives" deviceset="R-EU_" device="R0603" technology="0.082" value="82m"/>
 <part name="Q7" library="bschulz" deviceset="MOSFET-PCH" device="-AO3419" value="AO3419"/>
 <part name="Q3" library="bschulz" deviceset="MOSFET-NCH" device="-2N7002P" value="2N7002"/>
 <part name="R3" library="bschulz_passives" deviceset="R-EU_" device="R0402" technology="10K" value="10k"/>
 <part name="GND20" library="supply1" library_urn="urn:adsk.eagle:library:371" deviceset="GND" device=""/>
-<part name="R7" library="bschulz_passives" deviceset="R-EU_" device="R0603" value="82m"/>
+<part name="R7" library="bschulz_passives" deviceset="R-EU_" device="R0603" technology="0.082" value="82m"/>
 <part name="Q8" library="bschulz" deviceset="MOSFET-PCH" device="-AO3419" value="AO3419"/>
 <part name="Q4" library="bschulz" deviceset="MOSFET-NCH" device="-2N7002P" value="2N7002"/>
 <part name="R4" library="bschulz_passives" deviceset="R-EU_" device="R0402" technology="10K" value="10k"/>
 <part name="GND1" library="supply1" library_urn="urn:adsk.eagle:library:371" deviceset="GND" device=""/>
-<part name="R8" library="bschulz_passives" deviceset="R-EU_" device="R0603" value="82m"/>
+<part name="R8" library="bschulz_passives" deviceset="R-EU_" device="R0603" technology="0.082" value="82m"/>
 <part name="J1" library="GEMS_Plugs" deviceset="CONN_TALON" device="_REMOTE"/>
 <part name="GND5" library="supply1" library_urn="urn:adsk.eagle:library:371" deviceset="GND" device=""/>
@@
 <part name="GND24" library="supply1" library_urn="urn:adsk.eagle:library:371" deviceset="GND" device=""/>
 <part name="U8" library="bschulz" deviceset="MCP23018" device="QFN"/>
-<part name="R14" library="bschulz_passives" deviceset="R-EU_" device="R0603"/>
-<part name="R13" library="bschulz_passives" deviceset="R-EU_" device="R0603"/>
+<part name="R14" library="bschulz_passives" deviceset="R-EU_" device="R0603" technology="49.9K" value="49.9k"/>
+<part name="R13" library="bschulz_passives" deviceset="R-EU_" device="R0603" technology="110K" value="110k"/>
 <part name="GND44" library="supply1" library_urn="urn:adsk.eagle:library:371" deviceset="GND" device=""/>
 <part name="GND45" library="supply1" library_urn="urn:adsk.eagle:library:371" deviceset="GND" device=""/>
@@
 <part name="U7" library="bschulz" deviceset="24AA02" device="SOT23"/>
 <part name="GND56" library="supply1" library_urn="urn:adsk.eagle:library:371" deviceset="GND" device=""/>
-<part name="R16" library="bschulz_passives" deviceset="R-EU_" device="R0402"/>
-<part name="R15" library="bschulz_passives" deviceset="R-EU_" device="R0402"/>
+<part name="R16" library="bschulz_passives" deviceset="R-EU_" device="R0402" technology="10K" value="10k"/>
+<part name="R15" library="bschulz_passives" deviceset="R-EU_" device="R0402" technology="10K" value="10k"/>
 <part name="GND29" library="supply1" library_urn="urn:adsk.eagle:library:371" deviceset="GND" device=""/>
 <part name="U18" library="bschulz" deviceset="SN74AUP1G08" device="DCK"/>
@@
 <part name="R26" library="bschulz_passives" deviceset="R-EU_" device="R0402" technology="10K" value="10k"/>
 <part name="GND63" library="supply1" library_urn="urn:adsk.eagle:library:371" deviceset="GND" device=""/>
+<part name="TP1" library="bschulz" deviceset="TESTPOINT" device="RCU"/>
+<part name="TP2" library="bschulz" deviceset="TESTPOINT" device="RCU"/>
+<part name="TP3" library="bschulz" deviceset="TESTPOINT" device="RCU"/>
+<part name="TP4" library="bschulz" deviceset="TESTPOINT" device="RCU"/>
+<part name="TP5" library="bschulz" deviceset="TESTPOINT" device="RCU"/>
+<part name="TP6" library="bschulz" deviceset="TESTPOINT" device="RCU"/>
 </parts>
 <sheets>
@@
 <text x="124.46" y="157.48" size="1.778" layer="91" align="center">ALPHA</text>
 <text x="71.12" y="203.2" size="6.4516" layer="91">ADD DECOUPLING CAP!</text>
+<text x="170.18" y="58.42" size="6.4516" layer="91" align="center">Fix! </text>
+<text x="129.54" y="147.32" size="2.54" layer="91" align="center">ADR: 0x22</text>
 </plain>
 <instances>
@@
 <attribute name="NAME" x="62.0014" y="107.95" size="1.778" layer="95" rot="R90"/>
 <attribute name="VALUE" x="66.802" y="107.95" size="1.778" layer="96" rot="R90"/>
+</instance>
+<instance part="TP1" gate="G$1" x="68.58" y="73.66" smashed="yes" rot="R90">
+<attribute name="NAME" x="64.77" y="71.12" size="1.27" layer="95" rot="R180" align="center"/>
+</instance>
+<instance part="TP2" gate="G$1" x="68.58" y="68.58" smashed="yes" rot="R90">
+<attribute name="NAME" x="64.77" y="66.04" size="1.27" layer="95" rot="R180" align="center"/>
+</instance>
+<instance part="TP3" gate="G$1" x="68.58" y="63.5" smashed="yes" rot="R90">
+<attribute name="NAME" x="64.77" y="60.96" size="1.27" layer="95" rot="R180" align="center"/>
+</instance>
+<instance part="TP4" gate="G$1" x="68.58" y="58.42" smashed="yes" rot="R90">
+<attribute name="NAME" x="64.77" y="55.88" size="1.27" layer="95" rot="R180" align="center"/>
+</instance>
+<instance part="TP5" gate="G$1" x="68.58" y="53.34" smashed="yes" rot="R90">
+<attribute name="NAME" x="64.77" y="50.8" size="1.27" layer="95" rot="R180" align="center"/>
+</instance>
+<instance part="TP6" gate="G$1" x="68.58" y="48.26" smashed="yes" rot="R90">
+<attribute name="NAME" x="64.77" y="45.72" size="1.27" layer="95" rot="R180" align="center"/>
 </instance>
 </instances>
@@
 <pinref part="GND29" gate="1" pin="GND"/>
 </segment>
+<segment>
+<pinref part="TP1" gate="G$1" pin="P$1"/>
+<wire x1="68.58" y1="73.66" x2="73.66" y2="73.66" width="0.1524" layer="91"/>
+<label x="73.66" y="73.66" size="0.8128" layer="95" xref="yes"/>
+</segment>
 </net>
 <net name="SDA" class="0">
@@
 <label x="38.1" y="109.22" size="1.27" layer="95" xref="yes"/>
 </segment>
+<segment>
+<pinref part="TP2" gate="G$1" pin="P$1"/>
+<wire x1="68.58" y1="68.58" x2="73.66" y2="68.58" width="0.1524" layer="91"/>
+<label x="73.66" y="68.58" size="0.8128" layer="95" xref="yes"/>
+</segment>
 </net>
 <net name="SCL" class="0">
@@
 <wire x1="33.02" y1="111.76" x2="38.1" y2="111.76" width="0.1524" layer="91"/>
 <label x="38.1" y="111.76" size="1.27" layer="95" xref="yes"/>
+</segment>
+<segment>
+<pinref part="TP3" gate="G$1" pin="P$1"/>
+<wire x1="68.58" y1="63.5" x2="73.66" y2="63.5" width="0.1524" layer="91"/>
+<label x="73.66" y="63.5" size="0.8128" layer="95" xref="yes"/>
 </segment>
 </net>
@@
 <label x="38.1" y="114.3" size="1.27" layer="95" xref="yes"/>
 </segment>
+<segment>
+<pinref part="TP6" gate="G$1" pin="P$1"/>
+<wire x1="68.58" y1="48.26" x2="73.66" y2="48.26" width="0.1524" layer="91"/>
+<label x="73.66" y="48.26" size="0.8128" layer="95" xref="yes"/>
+</segment>
 </net>
 <net name="SDA_OB" class="0">
@@
 <label x="111.76" y="134.62" size="1.27" layer="95" rot="R180" xref="yes"/>
 </segment>
+<segment>
+<pinref part="TP4" gate="G$1" pin="P$1"/>
+<wire x1="68.58" y1="58.42" x2="73.66" y2="58.42" width="0.1524" layer="91"/>
+<label x="73.66" y="58.42" size="0.8128" layer="95" xref="yes"/>
+</segment>
 </net>
 <net name="SCL_OB" class="0">
@@
 <label x="111.76" y="132.08" size="1.27" layer="95" rot="R180" xref="yes"/>
 </segment>
-</net>
+<segment>
+<pinref part="TP5" gate="G$1" pin="P$1"/>
+<wire x1="68.58" y1="53.34" x2="73.66" y2="53.34" width="0.1524" layer="91"/>
+<label x="73.66" y="53.34" size="0.8128" layer="95" xref="yes"/>
+</segment>
+</net>
